Commit message: Change LIDAR position to get correct measurements

File: my_robot/urdf/my_robot.xacro (robot description, xacro)
@@ -173,5 +173,5 @@
   </link>
   <joint type="fixed" name="hokuyo_joint">
-    <origin xyz="0.15 0 0.1" rpy="0 0 0"/>
+    <origin xyz="0.2 0 0.13" rpy="0 0 0"/>
     <child link="hokuyo"/>
     <parent link="chassis"/>

Commit message: Adjust LIDAR position

File: my_robot/urdf/my_robot.xacro (robot description, xacro)
@@ -173,5 +173,5 @@
   </link>
   <joint type="fixed" name="hokuyo_joint">
-    <origin xyz="0.2 0 0.13" rpy="0 0 0"/>
+    <origin xyz="0.25 0 0.15" rpy="0 0 0"/>
     <child link="hokuyo"/>
     <parent link="chassis"/>
